File: FBG_PCB/FBG_PCB.kicad_pcb (KiCad board)
At the start: 2 copper layers, 37 parts, among them J1 Ground, J10 Pont diviseur Echo In 1-4, J11 17V, J12 17V, J13 Echo Out 5-8, J14 17V, J15 Buck converter 17V/5V, J16 Raspberry Power, J17 ES 5V + 5V, J18 5V, J19 5V, J2 Main switch + ES 17V, J20 5V, J21 5V, J3 Ground, J4 Ground, J5 Ground, J6 Echo Out 1-4, J7 Conn_01x02_Pin, J8 Vin 17V, J9 Pont diviseur Echo In 5-8

Commit message: Lot of new connectors
Parts:
- removed J3: Ground, Connector_Molex:Molex_SL_171971-0004_1x04_P2.54mm_Vertical
- added J22: Pont diviseur Echo In 1-4, Connector_Molex:Molex_SL_171971-0004_1x04_P2.54mm_Vertical, F.Cu at (134.6, 80.1)
- added J23: Pont diviseur Echo In 5-8, Connector_Molex:Molex_SL_171971-0004_1x04_P2.54mm_Vertical, F.Cu at (134.6, 88.8)
- added J24: Echo Out 1-4, Connector_Molex:Molex_SL_171971-0004_1x04_P2.54mm_Vertical, F.Cu at (134.6, 97.4)
- added J25: Echo Out 5-8, Connector_Molex:Molex_SL_171971-0004_1x04_P2.54mm_Vertical, F.Cu at (134.6, 106.0)
- added J26: Ground, Connector_Molex:Molex_SL_171971-0004_1x04_P2.54mm_Vertical, F.Cu at (68.4, 79.8)
- added J27: Ground, Connector_Molex:Molex_SL_171971-0004_1x04_P2.54mm_Vertical, F.Cu at (68.4, 88.4)
- added J28: Ground, Connector_Molex:Molex_SL_171971-0004_1x04_P2.54mm_Vertical, F.Cu at (68.4, 97.0)
- added J29: Ground, Connector_Molex:Molex_SL_171971-0004_1x04_P2.54mm_Vertical, F.Cu at (68.4, 105.7)
- added J30: Ground, Connector_Molex:Molex_SL_171971-0004_1x04_P2.54mm_Vertical, F.Cu at (68.4, 114.3)
- added J31: Ground, Connector_Molex:Molex_SL_171971-0004_1x04_P2.54mm_Vertical, F.Cu at (68.4, 123.0)
- J1: value Ground -> Vin 17V; footprint Connector_Molex:Molex_SL_171971-0004_1x04_P2.54mm_Vertical -> Connector_JST:JST_NV_B02P-NV_1x02_P5.00mm_Vertical
- J10: value Pont diviseur Echo In 1-4 -> Raspberry +17V switch
- J11: value 17V -> Buck converter 17V/5V
- J12: value 17V -> Raspberry Power+ 5V
- J13: value Echo Out 5-8 -> 17V
- J14: value 17V -> ES 5V + 5V
- J15: value Buck converter 17V/5V -> 5V
- J16: value Raspberry Power -> 5V
- J17: value ES 5V + 5V -> 5V
- J19: value 5V -> switch + ES 12V
- J2: value Main switch + ES 17V -> Vin 12V; footprint Connector_Molex:Molex_SL_171971-0004_1x04_P2.54mm_Vertical -> Connector_JST:JST_NV_B02P-NV_1x02_P5.00mm_Vertical
- J20, J21: value 5V -> 12V
- J6: value Echo Out 1-4 -> Ground
- J7: value Conn_01x02_Pin -> Ground; footprint Connector_JST:JST_NV_B02P-NV_1x02_P5.00mm_Vertical -> Connector_Molex:Molex_SL_171971-0004_1x04_P2.54mm_Vertical
- J8: value Vin 17V -> Ground; footprint Connector_JST:JST_NV_B02P-NV_1x02_P5.00mm_Vertical -> Connector_Molex:Molex_SL_171971-0004_1x04_P2.54mm_Vertical
- J9: value Pont diviseur Echo In 5-8 -> Ground
- moved J9 247.4 mm to (30.4, 183.5), turned to -90 degrees
- moved J6 212.2 mm to (56.4, 183.5), turned to -90 degrees
- moved J8 162.9 mm to (39.0, 183.5)
- moved J10 158.1 mm to (105.3, 114.7), turned to 0 degrees
- moved J13 138.9 mm to (119.9, 71.5)
- moved J1 118.7 mm to (17.2, 21.9), turned to 90 degrees
- moved J7 116.4 mm to (47.7, 183.5), turned to -90 degrees
- moved J11 107.0 mm to (105.3, 123.3)
- moved R4 106.5 mm to (194.0, 87.4), turned to 90 degrees
- moved R3 103.1 mm to (188.8, 87.4), turned to 90 degrees
- moved J20 102.9 mm to (134.6, 62.8)
- moved J21 102.9 mm to (134.6, 71.5)
- moved R2 100.2 mm to (183.7, 87.4), turned to 90 degrees
- moved R1 97.7 mm to (178.6, 87.4), turned to 90 degrees
- moved R6 93.7 mm to (184.0, 52.7), turned to 90 degrees
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Connections:
- J1 pad 2: Net-(J1-Pin_1) -> Net-(J1-Pin_2)
- J10 pad 1: Net-(J10-Pin_1) -> Net-(J1-Pin_1)
- J10 pad 3: Net-(J10-Pin_3) -> Net-(J10-Pin_2)
- J10 pad 4: Net-(J10-Pin_4) -> Net-(J10-Pin_2)
- J11 pad 2: Net-(J11-Pin_1) -> Net-(J11-Pin_2)
- J11 pad 3: Net-(J11-Pin_1) -> Net-(J1-Pin_2)
- J11 pad 4: Net-(J11-Pin_1) -> Net-(J10-Pin_2)
- J12 pad 1: Net-(J11-Pin_1) -> Net-(J11-Pin_2)
- J12 pad 2: Net-(J11-Pin_1) -> Net-(J11-Pin_2)
- J13 pad 1: Net-(J13-Pin_1) -> Net-(J10-Pin_2)
- J13 pad 2: Net-(J13-Pin_2) -> Net-(J10-Pin_2)
- J13 pad 3: Net-(J13-Pin_3) -> Net-(J10-Pin_2)
- J13 pad 4: Net-(J13-Pin_4) -> Net-(J10-Pin_2)
- J14 pad 1: Net-(J11-Pin_1) -> Net-(J14-Pin_1)
- J14 pad 2: Net-(J11-Pin_1) -> Net-(J14-Pin_1)
- J14 pad 3: Net-(J11-Pin_1) -> Net-(J14-Pin_1)
- J14 pad 4: Net-(J11-Pin_1) -> Net-(J11-Pin_2)
- J15 pad 1: Net-(J15-Pin_1) -> Net-(J14-Pin_1)
- J15 pad 2: Net-(J15-Pin_2) -> Net-(J14-Pin_1)
- J15 pad 3: Net-(J1-Pin_1) -> Net-(J14-Pin_1)
- J15 pad 4: Net-(J15-Pin_4) -> Net-(J14-Pin_1)
- J16 pad 1: Net-(J15-Pin_2) -> Net-(J14-Pin_1)
- J16 pad 2: Net-(J15-Pin_2) -> Net-(J14-Pin_1)
- J16 pad 3: Net-(J15-Pin_1) -> Net-(J14-Pin_1)
- J16 pad 4: Net-(J15-Pin_1) -> Net-(J14-Pin_1)
- J17 pad 1: Net-(J17-Pin_1) -> Net-(J14-Pin_1)
- J17 pad 2: Net-(J17-Pin_1) -> Net-(J14-Pin_1)
- J17 pad 3: Net-(J17-Pin_1) -> Net-(J14-Pin_1)
- J17 pad 4: Net-(J15-Pin_2) -> Net-(J14-Pin_1)
- J18 pad 1: Net-(J17-Pin_1) -> Net-(J14-Pin_1)
- J18 pad 2: Net-(J17-Pin_1) -> Net-(J14-Pin_1)
- J18 pad 3: Net-(J17-Pin_1) -> Net-(J14-Pin_1)
- J18 pad 4: Net-(J17-Pin_1) -> Net-(J14-Pin_1)
- J19 pad 1: Net-(J17-Pin_1) -> Net-(J19-Pin_1)
- J19 pad 2: Net-(J17-Pin_1) -> Net-(J19-Pin_2)
- J19 pad 3: Net-(J17-Pin_1) -> Net-(J19-Pin_2)
- J19 pad 4: Net-(J17-Pin_1) -> Net-(J19-Pin_4)
- J2 pad 1: Net-(J2-Pin_1) -> Net-(J19-Pin_4)
- J2 pad 2: Net-(J15-Pin_4) -> Net-(J1-Pin_2)
- J20 pad 1: Net-(J17-Pin_1) -> Net-(J19-Pin_1)
- J20 pad 2: Net-(J17-Pin_1) -> Net-(J19-Pin_1)
- J20 pad 3: Net-(J17-Pin_1) -> Net-(J19-Pin_1)
- J20 pad 4: Net-(J17-Pin_1) -> Net-(J19-Pin_1)
- J21 pad 1: Net-(J17-Pin_1) -> Net-(J19-Pin_1)
- J21 pad 2: Net-(J17-Pin_1) -> Net-(J19-Pin_1)
- J21 pad 3: Net-(J17-Pin_1) -> Net-(J19-Pin_1)
- J21 pad 4: Net-(J17-Pin_1) -> Net-(J19-Pin_1)
- J4 pad 1: Net-(J1-Pin_1) -> Net-(J1-Pin_2)
- J4 pad 2: Net-(J1-Pin_1) -> Net-(J1-Pin_2)
- J4 pad 3: Net-(J1-Pin_1) -> Net-(J1-Pin_2)
- J4 pad 4: Net-(J1-Pin_1) -> Net-(J1-Pin_2)
- J5 pad 1: Net-(J1-Pin_1) -> Net-(J1-Pin_2)
- J5 pad 2: Net-(J1-Pin_1) -> Net-(J1-Pin_2)
- J5 pad 3: Net-(J1-Pin_1) -> Net-(J1-Pin_2)
- J5 pad 4: Net-(J1-Pin_1) -> Net-(J1-Pin_2)
- J6 pad 1: Net-(J6-Pin_1) -> Net-(J1-Pin_2)
- J6 pad 2: Net-(J6-Pin_2) -> Net-(J1-Pin_2)
- J6 pad 3: Net-(J6-Pin_3) -> Net-(J1-Pin_2)
- J6 pad 4: Net-(J6-Pin_4) -> Net-(J1-Pin_2)
- J7 pad 1: unconnected-(J7-Pin_1-Pad1) -> Net-(J1-Pin_2)
- J7 pad 2: unconnected-(J7-Pin_2-Pad2) -> Net-(J1-Pin_2)
- J8 pad 1: Net-(J2-Pin_1) -> Net-(J1-Pin_2)
- J8 pad 2: Net-(J1-Pin_1) -> Net-(J1-Pin_2)
- J9 pad 1: Net-(J9-Pin_1) -> Net-(J1-Pin_2)
- J9 pad 2: Net-(J9-Pin_2) -> Net-(J1-Pin_2)
- J9 pad 3: Net-(J9-Pin_3) -> Net-(J1-Pin_2)
- J9 pad 4: Net-(J9-Pin_4) -> Net-(J1-Pin_2)
- R1 pad 1: Net-(J10-Pin_4) -> Net-(J22-Pin_4)
- R1 pad 2: Net-(J6-Pin_1) -> Net-(J24-Pin_1)
- R10 pad 1: Net-(J13-Pin_1) -> Net-(J23-Pin_3)
- R10 pad 2: Net-(J1-Pin_1) -> Net-(J25-Pin_2)
- R11 pad 1: Net-(J9-Pin_3) -> Net-(J23-Pin_2)
- R11 pad 2: Net-(J13-Pin_2) -> Net-(J25-Pin_3)
- R12 pad 1: Net-(J13-Pin_2) -> Net-(J23-Pin_1)
- R12 pad 2: Net-(J1-Pin_1) -> Net-(J25-Pin_4)
- R13 pad 1: Net-(J9-Pin_2) -> Net-(J25-Pin_1)
- R13 pad 2: Net-(J13-Pin_3) -> Net-(J1-Pin_2)
- R14 pad 1: Net-(J13-Pin_3) -> Net-(J25-Pin_2)
- R14 pad 2: Net-(J1-Pin_1) -> Net-(J1-Pin_2)
- R15 pad 1: Net-(J9-Pin_1) -> Net-(J25-Pin_3)
- R15 pad 2: Net-(J13-Pin_4) -> Net-(J1-Pin_2)
- R16 pad 1: Net-(J13-Pin_4) -> Net-(J25-Pin_4)
- R16 pad 2: Net-(J1-Pin_1) -> Net-(J1-Pin_2)
- R2 pad 1: Net-(J10-Pin_3) -> Net-(J22-Pin_3)
- R2 pad 2: Net-(J6-Pin_2) -> Net-(J24-Pin_2)
- R3 pad 1: Net-(J10-Pin_2) -> Net-(J22-Pin_2)
- R3 pad 2: Net-(J6-Pin_3) -> Net-(J24-Pin_3)
- R4 pad 1: Net-(J6-Pin_1) -> Net-(J22-Pin_1)
- R4 pad 2: Net-(J1-Pin_1) -> Net-(J24-Pin_4)
- R5 pad 1: Net-(J6-Pin_2) -> Net-(J24-Pin_1)
- R5 pad 2: Net-(J1-Pin_1) -> Net-(J1-Pin_2)
- R6 pad 1: Net-(J6-Pin_3) -> Net-(J24-Pin_2)
- R6 pad 2: Net-(J1-Pin_1) -> Net-(J1-Pin_2)
- R7 pad 1: Net-(J10-Pin_1) -> Net-(J24-Pin_3)
- R7 pad 2: Net-(J6-Pin_4) -> Net-(J1-Pin_2)
- R8 pad 1: Net-(J6-Pin_4) -> Net-(J24-Pin_4)
- R8 pad 2: Net-(J1-Pin_1) -> Net-(J1-Pin_2)
- R9 pad 1: Net-(J9-Pin_4) -> Net-(J23-Pin_4)
- R9 pad 2: Net-(J13-Pin_1) -> Net-(J25-Pin_1)
Routing:
- net Net-(J2-Pin_1): track 35.2 -> 0.00 mm

Commit message: trig + echo
Parts:
- J26: value Ground -> Control Driver Motor In
- J27: value Ground -> Control Driver Motor In +Out
- J28: value Ground -> Control Driver Motor Out
- J29: value Ground -> Trig In
- J30: value Ground -> Trig In + Out
- J31: value Ground -> Trig Out
- moved J8 43.4 mm to (82.5, 183.0), turned to 0 degrees
- moved J6 32.2 mm to (40.5, 155.5), turned to 0 degrees
- moved J9 21.4 mm to (24.0, 163.0)
- moved J4 20.0 mm to (90.0, 171.9), turned to 0 degrees
- moved J5 18.2 mm to (68.0, 165.5), turned to 0 degrees
- moved J7 17.2 mm to (64.9, 183.0), turned to 0 degrees
Connections:
- J26 pad 1: unconnected-(J26-Pin_1-Pad1) -> Net-(J26-Pin_1)
- J26 pad 2: unconnected-(J26-Pin_2-Pad2) -> Net-(J26-Pin_2)
- J26 pad 3: unconnected-(J26-Pin_3-Pad3) -> Net-(J26-Pin_3)
- J26 pad 4: unconnected-(J26-Pin_4-Pad4) -> Net-(J26-Pin_4)
- J27 pad 1: unconnected-(J27-Pin_1-Pad1) -> Net-(J27-Pin_1)
- J27 pad 2: unconnected-(J27-Pin_2-Pad2) -> Net-(J27-Pin_2)
- J27 pad 3: unconnected-(J27-Pin_3-Pad3) -> Net-(J27-Pin_2)
- J27 pad 4: unconnected-(J27-Pin_4-Pad4) -> Net-(J27-Pin_1)
- J28 pad 1: unconnected-(J28-Pin_1-Pad1) -> Net-(J26-Pin_1)
- J28 pad 2: unconnected-(J28-Pin_2-Pad2) -> Net-(J26-Pin_2)
- J28 pad 3: unconnected-(J28-Pin_3-Pad3) -> Net-(J26-Pin_3)
- J28 pad 4: unconnected-(J28-Pin_4-Pad4) -> Net-(J26-Pin_4)
- J29 pad 1: unconnected-(J29-Pin_1-Pad1) -> Net-(J29-Pin_1)
- J29 pad 2: unconnected-(J29-Pin_2-Pad2) -> Net-(J29-Pin_2)
- J29 pad 3: unconnected-(J29-Pin_3-Pad3) -> Net-(J29-Pin_3)
- J29 pad 4: unconnected-(J29-Pin_4-Pad4) -> Net-(J29-Pin_4)
- J30 pad 1: unconnected-(J30-Pin_1-Pad1) -> Net-(J30-Pin_1)
- J30 pad 2: unconnected-(J30-Pin_2-Pad2) -> Net-(J30-Pin_2)
- J30 pad 3: unconnected-(J30-Pin_3-Pad3) -> Net-(J30-Pin_2)
- J30 pad 4: unconnected-(J30-Pin_4-Pad4) -> Net-(J30-Pin_1)
- J31 pad 1: unconnected-(J31-Pin_1-Pad1) -> Net-(J29-Pin_1)
- J31 pad 2: unconnected-(J31-Pin_2-Pad2) -> Net-(J29-Pin_2)
- J31 pad 3: unconnected-(J31-Pin_3-Pad3) -> Net-(J29-Pin_3)
- J31 pad 4: unconnected-(J31-Pin_4-Pad4) -> Net-(J29-Pin_4)
- R1 pad 2: Net-(J24-Pin_1) -> Net-(J24-Pin_4)
- R10 pad 2: Net-(J25-Pin_2) -> Net-(J25-Pin_3)
- R11 pad 2: Net-(J25-Pin_3) -> Net-(J25-Pin_2)
- R12 pad 2: Net-(J25-Pin_4) -> Net-(J25-Pin_1)
- R13 pad 1: Net-(J25-Pin_1) -> Net-(J25-Pin_4)
- R14 pad 1: Net-(J25-Pin_2) -> Net-(J25-Pin_3)
- R15 pad 1: Net-(J25-Pin_3) -> Net-(J25-Pin_2)
- R16 pad 1: Net-(J25-Pin_4) -> Net-(J25-Pin_1)
- R2 pad 2: Net-(J24-Pin_2) -> Net-(J24-Pin_3)
- R3 pad 2: Net-(J24-Pin_3) -> Net-(J24-Pin_2)
- R4 pad 2: Net-(J24-Pin_4) -> Net-(J24-Pin_1)
- R5 pad 1: Net-(J24-Pin_1) -> Net-(J24-Pin_4)
- R6 pad 1: Net-(J24-Pin_2) -> Net-(J24-Pin_3)
- R7 pad 1: Net-(J24-Pin_3) -> Net-(J24-Pin_2)
- R8 pad 1: Net-(J24-Pin_4) -> Net-(J24-Pin_1)
- R9 pad 2: Net-(J25-Pin_1) -> Net-(J25-Pin_4)

Commit message: V1
Parts:
- added J32: I2C Out, Connector_Molex:Molex_SL_171971-0004_1x04_P2.54mm_Vertical, F.Cu at (143.2, -189.0)
- added J33: I2C SCL In, Connector_Molex:Molex_SL_171971-0004_1x04_P2.54mm_Vertical, F.Cu at (151.0, -149.9)
- added J34: I2C SCL In +SDA In, Connector_Molex:Molex_SL_171971-0004_1x04_P2.54mm_Vertical, F.Cu at (151.0, -132.9)
- added J35: I2C SDA In, Connector_Molex:Molex_SL_171971-0004_1x04_P2.54mm_Vertical, F.Cu at (151.0, -116.5)
- added J36: Control Motor CanLift Out +In, Connector_Molex:Molex_SL_171971-0004_1x04_P2.54mm_Vertical, F.Cu at (139.2, -117.0)
- added J37: Encoder M1 +M2 Out, Connector_Molex:Molex_SL_171971-0004_1x04_P2.54mm_Vertical, F.Cu at (124.0, -117.0)
- added J38: Encoder M1 +M2 In, Connector_Molex:Molex_SL_171971-0004_1x04_P2.54mm_Vertical, F.Cu at (111.0, -117.0)
- added J39: Bonus Out, Connector_Molex:Molex_SL_171971-0004_1x04_P2.54mm_Vertical, F.Cu at (116.0, -158.0)
- added J40: Bonus In, Connector_Molex:Molex_SL_171971-0004_1x04_P2.54mm_Vertical, F.Cu at (124.9, -171.5)
- added J41: Bonus Out, Connector_Molex:Molex_SL_171971-0004_1x04_P2.54mm_Vertical, F.Cu at (131.3, -158.0)
- added J42: Bonus In, Connector_Molex:Molex_SL_171971-0004_1x04_P2.54mm_Vertical, F.Cu at (139.7, -171.5)
- J22: value Pont diviseur Echo In 1-4 -> Pont diviseur Echo Out 1-4
- J23: value Pont diviseur Echo In 5-8 -> Pont diviseur Echo Out 5-8
- J24: value Echo Out 1-4 -> Echo In 1-4
- J25: value Echo Out 5-8 -> Echo In 5-8
- J26: value Control Driver Motor In -> Control Driver Motor Out
- J27: value Control Driver Motor In +Out -> Control Driver Motor Out + Trig Out
- J28: value Control Driver Motor Out -> Control Driver Motor In
- J30: value Trig In + Out -> Control Driver Motor In + Trig In
- R1, R10, R11, R12, R13, R14, R15, R16, R2, R3, R4, R5, R6, R7, R8, R9: footprint Resistor_THT:R_Axial_DIN0411_L9.9mm_D3.6mm_P25.40mm_Horizontal -> Resistor_THT:R_Axial_DIN0207_L6.3mm_D2.5mm_P10.16mm_Horizontal
- moved J31 312.7 mm to (89.5, -189.0)
- moved J25 295.2 mm to (125.3, -189.0)
- moved J9 294.0 mm to (145.4, -104.8), turned to 0 degrees
- moved J7 291.5 mm to (111.6, -104.8)
- moved J8 291.4 mm to (128.6, -104.8)
- moved J24 287.7 mm to (107.4, -189.0)
- moved J30 286.5 mm to (87.6, -171.5)
- moved J11 281.0 mm to (35.9, -149.0), turned to 90 degrees
- moved J29 279.7 mm to (105.8, -171.5)
- moved J4 278.6 mm to (57.4, -104.8)
- moved J27 277.4 mm to (71.5, -189.0)
- moved R13 276.0 mm to (91.1, -143.0), turned to 180 degrees
- moved J5 270.4 mm to (75.6, -104.8)
- moved R14 270.0 mm to (91.1, -139.0), turned to 180 degrees
- moved J26 269.2 mm to (53.6, -189.0)
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Connections:
- J11 pad 1: Net-(J11-Pin_1) -> Net-(J10-Pin_2)
- J11 pad 2: Net-(J11-Pin_2) -> Net-(J1-Pin_2)
- J11 pad 3: Net-(J1-Pin_2) -> Net-(J11-Pin_3)
- J11 pad 4: Net-(J10-Pin_2) -> Net-(J11-Pin_4)
- J12 pad 1: Net-(J11-Pin_2) -> Net-(J11-Pin_3)
- J12 pad 2: Net-(J11-Pin_2) -> Net-(J11-Pin_3)
- J12 pad 3: Net-(J11-Pin_1) -> Net-(J11-Pin_4)
- J12 pad 4: Net-(J11-Pin_1) -> Net-(J11-Pin_4)
- J14 pad 4: Net-(J11-Pin_2) -> Net-(J11-Pin_3)
- J27 pad 3: Net-(J27-Pin_2) -> Net-(J27-Pin_3)
- J27 pad 4: Net-(J27-Pin_1) -> Net-(J27-Pin_4)
- J30 pad 1: Net-(J30-Pin_1) -> Net-(J27-Pin_1)
- J30 pad 2: Net-(J30-Pin_2) -> Net-(J27-Pin_2)
- J30 pad 3: Net-(J30-Pin_2) -> Net-(J27-Pin_3)
- J30 pad 4: Net-(J30-Pin_1) -> Net-(J27-Pin_4)
- R1 pad 1: Net-(J22-Pin_4) -> Net-(J22-Pin_1)
- R1 pad 2: Net-(J24-Pin_4) -> Net-(J24-Pin_1)
- R10 pad 1: Net-(J23-Pin_3) -> Net-(J23-Pin_2)
- R10 pad 2: Net-(J25-Pin_3) -> Net-(J25-Pin_2)
- R11 pad 1: Net-(J23-Pin_2) -> Net-(J23-Pin_3)
- R11 pad 2: Net-(J25-Pin_2) -> Net-(J25-Pin_3)
- R12 pad 1: Net-(J23-Pin_1) -> Net-(J23-Pin_4)
- R12 pad 2: Net-(J25-Pin_1) -> Net-(J25-Pin_4)
- R13 pad 1: Net-(J25-Pin_4) -> Net-(J25-Pin_1)
- R14 pad 1: Net-(J25-Pin_3) -> Net-(J25-Pin_2)
- R15 pad 1: Net-(J25-Pin_2) -> Net-(J25-Pin_3)
- R16 pad 1: Net-(J25-Pin_1) -> Net-(J25-Pin_4)
- R2 pad 1: Net-(J22-Pin_3) -> Net-(J22-Pin_2)
- R2 pad 2: Net-(J24-Pin_3) -> Net-(J24-Pin_2)
- R3 pad 1: Net-(J22-Pin_2) -> Net-(J22-Pin_3)
- R3 pad 2: Net-(J24-Pin_2) -> Net-(J24-Pin_3)
- R4 pad 1: Net-(J22-Pin_1) -> Net-(J22-Pin_4)
- R4 pad 2: Net-(J24-Pin_1) -> Net-(J24-Pin_4)
- R5 pad 1: Net-(J24-Pin_4) -> Net-(J24-Pin_1)
- R6 pad 1: Net-(J24-Pin_3) -> Net-(J24-Pin_2)
- R7 pad 1: Net-(J24-Pin_2) -> Net-(J24-Pin_3)
- R8 pad 1: Net-(J24-Pin_1) -> Net-(J24-Pin_4)
- R9 pad 1: Net-(J23-Pin_4) -> Net-(J23-Pin_1)
- R9 pad 2: Net-(J25-Pin_4) -> Net-(J25-Pin_1)
Routing:
- net Net-(J1-Pin_2): track 0.00 -> 226.1 mm
- net Net-(J14-Pin_1): track 0.00 -> 94.2 mm
- net Net-(J32-Pin_3): track 0.00 -> 80.1 mm
- net Net-(J25-Pin_4): track 0.00 -> 79.4 mm
- net Net-(J25-Pin_3): track 0.00 -> 73.8 mm
- net Net-(J25-Pin_2): track 0.00 -> 70.2 mm
- net Net-(J25-Pin_1): track 0.00 -> 65.3 mm
- net Net-(J32-Pin_1): track 0.00 -> 63.3 mm
- net Net-(J24-Pin_4): track 0.00 -> 53.9 mm
- net Net-(J10-Pin_2): track 0.00 -> 53.4 mm, vias 0 -> 1
- net Net-(J24-Pin_3): track 0.00 -> 48.9 mm
- net Net-(J24-Pin_2): track 0.00 -> 43.8 mm
- net Net-(J24-Pin_1): track 0.00 -> 39.3 mm
- net Net-(J11-Pin_4): track 0.00 -> 37.0 mm
- net Net-(J23-Pin_1): track 0.00 -> 36.9 mm
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Other:
- board outline added: 128 x 96 mm
- copper layers 2 -> 4
- board text added: "1 2"
- board text added: "1 2 3 4"
- board text added: "12V"
- board text added: "4 3 2 1"
- board text added: "5V"
- board text added: "EUROBOT 2025 FBG Team"
- board text added: "GND"
- board text added: "Raspberry Interface"

Commit message: V2
Parts:
- J10: value Raspberry +17V switch -> Raspberry switch
- J11: value Buck converter 17V/5V -> Buck converter
- J12: value Raspberry Power+ 5V -> Raspberry Power
- J14: value ES 5V + 5V -> ES 5V
- J19: value switch + ES 12V -> switch + ES
- J22: value Pont diviseur Echo Out 1-4 -> Echo Out 1-4
- J23: value Pont diviseur Echo Out 5-8 -> Echo Out 5-8
- J26: value Control Driver Motor Out -> Driver Motor Out
- J27: value Control Driver Motor Out + Trig Out -> Driver Motor Out + Trig Out
- J28: value Control Driver Motor In -> Driver Motor In
- J30: value Control Driver Motor In + Trig In -> Driver Motor In + Trig In
- J36: value Control Motor CanLift Out +In -> Motor CanLift Out +In
- moved J37 254.2 mm to (366.0, -194.7), turned to 0 degrees
- moved J38 246.3 mm to (350.4, -175.0), turned to 0 degrees
- moved J36 238.5 mm to (372.0, -169.2)
- moved J41 225.4 mm to (353.5, -120.2), turned to 90 degrees
- moved J35 223.9 mm to (372.0, -152.2)
- moved J33 223.0 mm to (372.0, -120.0)
- moved J22 222.0 mm to (340.0, -147.1)
- moved J23 222.0 mm to (355.0, -147.1)
- moved J34 221.0 mm to (372.0, -135.9)
- moved J9 220.4 mm to (365.8, -107.8)
- moved J8 216.9 mm to (345.5, -107.8)
- moved J39 215.4 mm to (331.4, -161.0)
- moved J7 213.7 mm to (325.2, -107.8)
- moved J21 213.5 mm to (313.0, -120.0)
- moved R1 212.4 mm to (317.1, -162.3)
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Routing:
- net Net-(J32-Pin_1): track 63.3 -> 86.4 mm
- net Net-(J32-Pin_3): track 80.1 -> 63.8 mm
- net Net-(J1-Pin_2): track 226.1 -> 242.4 mm
- net Net-(J37-Pin_4): track 13.0 -> 26.2 mm
- net Net-(J37-Pin_3): track 13.0 -> 26.2 mm
- net Net-(J37-Pin_2): track 13.0 -> 26.2 mm
- net Net-(J37-Pin_1): track 13.0 -> 26.2 mm
- net Net-(J23-Pin_1): track 36.9 -> 49.1 mm
- net Net-(J23-Pin_2): track 35.0 -> 45.9 mm
- net Net-(J23-Pin_3): track 33.1 -> 43.7 mm
- net Net-(J23-Pin_4): track 31.2 -> 41.9 mm
- net Net-(J22-Pin_1): track 19.2 -> 29.6 mm
- net Net-(J22-Pin_2): track 18.3 -> 28.5 mm
- net Net-(J22-Pin_3): track 17.7 -> 27.9 mm
- net Net-(J22-Pin_4): track 17.1 -> 27.3 mm
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Other:
- board size 128 x 96 mm -> 150 x 100 mm
