File: FBG_PCB/FBG_PCB.kicad_pcb (KiCad board)
At the start: 4 copper layers, 150 x 100 mm, 57 parts, among them J1 Vin 17V, J10 Raspberry switch, J11 Buck converter, J12 Raspberry Power, J13 17V, J14 ES 5V, J15 5V, J16 5V, J17 5V, J18 5V, J19 switch + ES, J2 Vin 12V, J20 12V, J21 12V, J22 Echo Out 1-4, J23 Echo Out 5-8, J24 Echo In 1-4, J25 Echo In 5-8, J26 Driver Motor Out, J27 Driver Motor Out + Trig Out, J28 Driver Motor In, J29 Trig In, J30 Driver Motor In + Trig In, J31 Trig Out, J32 I2C Out, J33 I2C SCL In, J34 I2C SCL In +SDA In, J35 I2C SDA In, J36 Motor CanLift Out +In, J37 Encoder M1 +M2 Out, J38 Encoder M1 +M2 In, J39 Bonus Out, J4 Ground, J40 Bonus In, J41 Bonus Out, J42 Bonus In, J5 Ground, J6 Ground, J7 Ground, J8 Ground, J9 Ground

Commit message: V2.1
Parts:
- moved J38 3.01 mm to (347.4, -175.0)
- moved J29 2.93 mm to (310.1, -175.0)
- moved J40 2.76 mm to (328.7, -175.0)
- moved J39 2.65 mm to (328.7, -161.0)
- moved J30 2.54 mm to (291.5, -175.0)
- moved J28 2.15 mm to (272.8, -175.0)
- moved J13 1.77 mm to (254.2, -175.0)
Routing:
- net Net-(J10-Pin_2): track 55.8 -> 52.1 mm
- net Net-(J29-Pin_3): track 30.4 -> 27.4 mm
- net Net-(J29-Pin_2): track 31.1 -> 28.1 mm
- net Net-(J29-Pin_4): track 30.4 -> 27.4 mm
- net Net-(J26-Pin_2): track 29.6 -> 27.4 mm
- net Net-(J26-Pin_4): track 29.6 -> 27.4 mm
- net Net-(J26-Pin_3): track 29.6 -> 27.4 mm
- net Net-(J27-Pin_1): track 30.0 -> 27.9 mm
- net Net-(J27-Pin_3): track 30.0 -> 28.1 mm
- net Net-(J27-Pin_4): track 30.0 -> 28.1 mm
- net Net-(J27-Pin_2): track 30.0 -> 28.1 mm
- net Net-(J29-Pin_1): track 29.7 -> 27.9 mm
- net Net-(J26-Pin_1): track 29.0 -> 27.4 mm
- net Net-(J37-Pin_4): track 26.2 -> 27.4 mm
- net Net-(J37-Pin_3): track 26.2 -> 27.4 mm
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